File: file/pcb/v2/4x6/TPS/TPS.kicad_sch (KiCad schematic)
At the start: 91 parts, among them J1 I2C, J2 FFC-0.5mm, 12p, J3 FFC-0.5mm, 12p, J4 PH2.0-2pin, J5 FFC-0.5mm, 6p, J6 FFC-0.5mm, 6p, K1 SW_Push, K10 SW_Push, K11 SW_Push, K12 SW_Push, K13 SW_Push, K14 SW_Push, K15 SW_Push, K16 SW_Push, K17 SW_Push, K18 SW_Push, K19 SW_Push, K2 SW_Push, K20 SW_Push, K21 SW_Push, K22 SW_Push, K23 SW_Push, K24 SW_Push, K25 EC-11, K3 SW_Push, K4 SW_Push, K5 SW_Push, K6 SW_Push, K7 SW_Push, K8 SW_Push, K9 SW_Push, SW1 SW_Push, SW2 MSKT-12D14, SW3 MSKT-12D14, T1 AudioJack4, U1 MCU_ProMicro_13p

Commit message: fix TRRS TX/RX pins
Parts:
- removed T1: AudioJack4, DreaM117er-keebLibrary:TRRS-PJ-320A, dual side x2, symbol DreaM117er_Library:TRRS
- added J9: AudioJack4, DreaM117er-keebLibrary:TRRS-PJ-320A, dual side x2, symbol Connector_Audio:AudioJack4
Connections:
- net GND: now also J9.S
- net TX: now also J9.R1
- net at F1.2, F2.2, JP15.2 (B)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: now also J9.T
- net at JP13.2 (B), JP14.2 (B): now also J9.R2
Changed lines of the file:
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@@
+	)
+	(symbol
+		(lib_id "Connector_Audio:AudioJack4")
+		(at 171.45 130.81 180)
+		(unit 1)
+		(exclude_from_sim no)
+		(in_bom yes)
+		(on_board yes)
+		(dnp no)
+		(fields_autoplaced yes)
+		(property "Reference" "J9"
+			(at 180.34 127.6349 0)
+			(effects
+				(font
+					(size 1.27 1.27)
+				)
+				(justify right)
+			)
+		)
+		(property "Value" "AudioJack4"
+			(at 180.34 130.1749 0)
+			(effects
+				(font
+					(size 1.27 1.27)
+				)
+				(justify right)
+			)
+		)
+		(property "Footprint" "DreaM117er-keebLibrary:TRRS-PJ-320A, dual side x2"
+			(at 171.45 130.81 0)
+			(effects
+				(font
+					(size 1.27 1.27)
+				)
+				(hide yes)
+			)
+		)
+		(property "Datasheet" "~"
+			(at 171.45 130.81 0)
+			(effects
+				(font
+					(size 1.27 1.27)
+				)
+				(hide yes)
+			)
+		)
+		(property "Description" "Audio Jack, 4 Poles (TRRS)"
+			(at 171.45 130.81 0)
+			(effects
+				(font
+					(size 1.27 1.27)
+				)
+				(hide yes)
+			)
+		)
+		(pin "S"
+		)
+		(pin "T"
+		)
+		(pin "R2"
+		)
+		(pin "R1"
+		)
+		(instances
+			(project ""
+				(path "/362e52b9-ba3a-40a2-a3a5-9227c3d95473"
+					(reference "J9")
+					(unit 1)
+				)
+			)
+		)
 	)
 	(symbol
@@
 					(unit 1)
 				)
-			)
-		)
-	)
-	(symbol
-		(lib_id "DreaM117er_Library:TRRS")
-		(at 175.26 135.89 0)
-		(unit 1)
-		(exclude_from_sim no)
-		(in_bom yes)
-		(on_board yes)
-		(dnp no)
-		(fields_autoplaced yes)
-		(property "Reference" "T1"
-			(at 180.975 128.27 0)
-			(effects
-				(font
-					(size 1.27 1.27)
-				)
-				(justify left)
-			)
-		)
-		(property "Value" "AudioJack4"
-			(at 180.975 130.81 0)
-			(effects
-				(font
-					(size 1.27 1.27)
-				)
-				(justify left)
-			)
-		)
-		(property "Footprint" "DreaM117er-keebLibrary:TRRS-PJ-320A, dual side x2"
-			(at 175.26 139.7 0)
-			(effects
-				(font
-					(size 1.524 1.524)
-				)
-				(hide yes)
-			)
-		)
-		(property "Datasheet" "~"
-			(at 175.26 137.16 0)
-			(effects
-				(font
-					(size 1.524 1.524)
-				)
-				(hide yes)
-			)
-		)
-		(property "Description" ""
-			(at 175.26 135.89 0)
-			(effects
-				(font
-					(size 1.27 1.27)
-				)
-			)
-		)
-		(pin "1"
-		)
-		(pin "2"
-		)
-		(pin "3"
-		)
-		(pin "4"
-		)
-		(instances
-			(project "TPS"
-				(path "/362e52b9-ba3a-40a2-a3a5-9227c3d95473"
-					(reference "T1")
-					(unit 1)
-				)

Commit message: fix main PCB file UI
Parts:
- J9: footprint DreaM117er-keebLibrary:TRRS-PJ-320A, dual side x2 -> DreaM117er-keebLibrary:TRRS-PJ-320A, dual side x2_3rd
Connections:
- net N/A1: now reaches SW2.3 (C)
- net row4: now reaches U1.9 (5/PC6)
- net N/A2: now reaches SW3.3 (C)
- no-connect marks 23 -> 20
Changed lines of the file:
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@@
 	)
 	(no_connect
-		(at 129.54 53.34)
-	)
-	(no_connect
 		(at 38.1 146.05)
 	)
@@
 	)
 	(no_connect
-		(at 218.44 96.52)
-	)
-	(no_connect
-		(at 218.44 78.74)
-	)
-	(no_connect
 		(at 38.1 138.43)
 	)
@@
 		)
 	)
+	(global_label "N{slash}A1"
+		(shape input)
+		(at 218.44 78.74 180)
+		(fields_autoplaced yes)
+		(effects
+			(font
+				(size 1.27 1.27)
+			)
+			(justify right)
+		)
+		(property "Intersheetrefs" "${INTERSHEET_REFS}"
+			(at 210.4957 78.74 0)
+			(effects
+				(font
+					(size 1.27 1.27)
+				)
+				(justify right)
+				(hide yes)
+			)
+		)
+	)
 	(global_label "col4"
 		(shape input)
@@
 		)
 	)
+	(global_label "N{slash}A2"
+		(shape input)
+		(at 218.44 96.52 180)
+		(fields_autoplaced yes)
+		(effects
+			(font
+				(size 1.27 1.27)
+			)
+			(justify right)
+		)
+		(property "Intersheetrefs" "${INTERSHEET_REFS}"
+			(at 210.4957 96.52 0)
+			(effects
+				(font
+					(size 1.27 1.27)
+				)
+				(justify right)
+				(hide yes)
+			)
+		)
+	)
 	(global_label "BAT+"
 		(shape input)
@@
 		)
 	)
+	(global_label "row4"
+		(shape input)
+		(at 129.54 53.34 180)
+		(fields_autoplaced yes)
+		(effects
+			(font
+				(size 1.27 1.27)
+			)
+			(justify right)
+		)
+		(property "Intersheetrefs" "${INTERSHEET_REFS}"
+			(at 122.0796 53.34 0)
+			(effects
+				(font
+					(size 1.27 1.27)
+				)
+				(justify right)
+				(hide yes)
+			)
+		)
+	)
 	(global_label "row0"
 		(shape input)
@@
 			)
 		)
-		(property "Footprint" "DreaM117er-keebLibrary:TRRS-PJ-320A, dual side x2"
+		(property "Footprint" "DreaM117er-keebLibrary:TRRS-PJ-320A, dual side x2_3rd"
 			(at 171.45 130.81 0)
 			(effects
